File: usbhub.brd (EAGLE design)
At the start: 0 parts

Commit message: aggiornamento pre stampa
Routing:
- net S$8: track 106.9 -> 208.5 mm, vias 4 -> 12
Changed lines of the file:
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@@
 <wire x1="43.18" y1="10.16" x2="48.26" y2="10.16" width="2.032" layer="1"/>
 <wire x1="53.34" y1="10.16" x2="48.26" y2="10.16" width="2.032" layer="1"/>
+<via x="26.67" y="77.47" extent="1-16" drill="1.524" diameter="2.54"/>
+<via x="31.75" y="77.47" extent="1-16" drill="1.524" diameter="2.54"/>
+<via x="36.83" y="77.47" extent="1-16" drill="1.524" diameter="2.54"/>
+<via x="41.91" y="77.47" extent="1-16" drill="1.524" diameter="2.54"/>
+<via x="46.99" y="77.47" extent="1-16" drill="1.524" diameter="2.54"/>
+<via x="52.07" y="77.47" extent="1-16" drill="1.524" diameter="2.54"/>
+<via x="57.15" y="77.47" extent="1-16" drill="1.524" diameter="2.54"/>
+<via x="62.23" y="77.47" extent="1-16" drill="1.524" diameter="2.54"/>
+<wire x1="26.67" y1="77.47" x2="26.67" y2="72.39" width="2.1844" layer="1"/>
+<wire x1="26.67" y1="72.39" x2="36.83" y2="72.39" width="2.1844" layer="1"/>
+<wire x1="36.83" y1="72.39" x2="46.99" y2="72.39" width="2.1844" layer="1"/>
+<wire x1="46.99" y1="72.39" x2="57.15" y2="72.39" width="2.1844" layer="1"/>
+<wire x1="57.15" y1="72.39" x2="57.15" y2="77.47" width="2.1844" layer="1"/>
+<wire x1="36.83" y1="77.47" x2="36.83" y2="72.39" width="2.1844" layer="1"/>
+<wire x1="46.99" y1="77.47" x2="46.99" y2="72.39" width="2.1844" layer="1"/>
+<wire x1="31.75" y1="77.47" x2="31.75" y2="82.55" width="2.1844" layer="1"/>
+<wire x1="31.75" y1="82.55" x2="41.91" y2="82.55" width="2.1844" layer="1"/>
+<wire x1="41.91" y1="82.55" x2="52.07" y2="82.55" width="2.1844" layer="1"/>
+<wire x1="52.07" y1="82.55" x2="62.23" y2="82.55" width="2.1844" layer="1"/>
+<wire x1="62.23" y1="82.55" x2="62.23" y2="77.47" width="2.1844" layer="1"/>
+<wire x1="41.91" y1="77.47" x2="41.91" y2="82.55" width="2.1844" layer="1"/>
+<wire x1="52.07" y1="77.47" x2="52.07" y2="82.55" width="2.1844" layer="1"/>
 </signal>
 <signal name="S$9">
